File: kicad_led_torch.kicad_pcb (KiCad board)
At the start: 2 copper layers, 4 parts, among them SW1 SW_DPST_x2

Commit message: Lunch break finish
Parts:
- added REF**: KiCad-Logo2_5mm_SilkScreen, Symbol:KiCad-Logo2_5mm_SilkScreen, B.Cu at (164.5, 94.0)
- moved D1 34.9 mm to (121.3, 94.0), turned to 180 degrees
- moved R1 25.5 mm to (125.1, 91.4), turned to -90 degrees
- moved BT1 17.6 mm to (164.5, 94.0)
- moved SW1 14.3 mm to (135.5, 97.2), turned to 90 degrees
Routing:
- net /LED_cathode: track 0.00 -> 65.2 mm
- net /bat_pos: track 0.00 -> 19.2 mm
- net Net-(SW1A-A): track 0.00 -> 17.2 mm
- net /LED_anode: track 0.00 -> 7.40 mm
Other:
- board outline added: 67.3 x 24.4 mm
- board text added: "+"
- board text added: "-"
- board text added: "v1.0"
